Commit message: Add link 3 to simple urdf

File: simple.urdf (robot description, URDF)
Before this commit: robot simple, 3 links, 2 joints
Links:
- added link link3, mass 0.4404689720232285; collision mesh filename=meshes/link3.stl scale=0.001 0.001 0.001; visual mesh filename=meshes/link3.stl scale=0.001 0.001 0.001
Joints:
- added joint joint3: type continuous, parent link2, child link3, origin xyz=0.00025 0.014791 0.108347 rpy=0 0 0, axis 1.0 0.0 0.0
